File: pcb/ESP-32-DSP_board/_autosave-ESP-32-DSP_board.kicad_sch (KiCad schematic)
At the start: 84 parts, among them J1 USB_C_Receptacle_USB2.0, J12 Conn_Coaxial, J2 Conn_01x10_Pin, J4 Conn_01x08_Pin, J5 SD_Card, J6 Conn_01x08_Pin, J7 Conn_01x08_Pin, J8 AudioJack3, U1 AZ1117IH-3.3, U2 AD5689BRUZ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

Commit message: ESP32-S3 DSP board
Parts:
- J12: footprint Connector_Coaxial:U.FL_Hirose_U.FL-R-SMT-1_Vertical -> RF_Antenna:Texas_SWRA117D_2.4GHz_Right
Changed lines of the file:
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@@
       (effects (font (size 1.27 1.27)) (justify left))
     )
-    (property "Footprint" "Connector_Coaxial:U.FL_Hirose_U.FL-R-SMT-1_Vertical" (at 55.245 114.3 0)
+    (property "Footprint" "RF_Antenna:Texas_SWRA117D_2.4GHz_Right" (at 55.245 114.3 0)
       (effects (font (size 1.27 1.27)) hide)
     )
