File: pcb/ESP-32-DSP_board/ESP-32-DSP_board.kicad_sch (KiCad schematic)
At the start: 84 parts, among them J1 USB_C_Receptacle_USB2.0, J12 Conn_Coaxial, J2 Conn_01x10_Pin, J4 Conn_01x08_Pin, J5 SD_Card, J6 Conn_01x08_Pin, J7 Conn_01x08_Pin, J8 AudioJack3, U1 AZ1117IH-3.3, U2 AD5689BRUZ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

Commit message: Added local pcb modifications
Parts:
- C1: footprint Capacitor_SMD:C_0402_1005Metric -> Capacitor_SMD:C_0805_2012Metric
- C37, C9: footprint Capacitor_SMD:C_0603_1608Metric -> Capacitor_SMD:C_0402_1005Metric
- J12: footprint Connector_Coaxial:U.FL_Hirose_U.FL-R-SMT-1_Vertical -> RF_Antenna:Texas_SWRA117D_2.4GHz_Right
- J8: footprint Connector_Audio:Jack_3.5mm_Switronic_ST-005-G_horizontal -> Connector_Audio:Jack_3.5mm_CUI_SJ-3523-SMT_Horizontal
Changed lines of the file:
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@@
       (effects (font (size 1.27 1.27)) (justify left))
     )
-    (property "Footprint" "Connector_Coaxial:U.FL_Hirose_U.FL-R-SMT-1_Vertical" (at 55.245 114.3 0)
+    (property "Footprint" "RF_Antenna:Texas_SWRA117D_2.4GHz_Right" (at 55.245 114.3 0)
       (effects (font (size 1.27 1.27)) hide)
     )
@@
       (effects (font (size 1.27 1.27)) (justify left))
     )
-    (property "Footprint" "Capacitor_SMD:C_0603_1608Metric" (at 360.3752 193.675 0)
+    (property "Footprint" "Capacitor_SMD:C_0402_1005Metric" (at 360.3752 193.675 0)
       (effects (font (size 1.27 1.27)) hide)
     )
@@
       (effects (font (size 1.27 1.27)) (justify left))
     )
-    (property "Footprint" "Capacitor_SMD:C_0402_1005Metric" (at 148.9202 44.45 0)
+    (property "Footprint" "Capacitor_SMD:C_0805_2012Metric" (at 148.9202 44.45 0)
       (effects (font (size 1.27 1.27)) hide)
     )
@@
       (effects (font (size 1.27 1.27)) (justify right))
     )
-    (property "Footprint" "Connector_Audio:Jack_3.5mm_Switronic_ST-005-G_horizontal" (at 376.555 214.63 0)
+    (property "Footprint" "Connector_Audio:Jack_3.5mm_CUI_SJ-3523-SMT_Horizontal" (at 376.555 214.63 0)
       (effects (font (size 1.27 1.27)) hide)
     )
@@
       (effects (font (size 1.27 1.27)) (justify left))
     )
-    (property "Footprint" "Capacitor_SMD:C_0603_1608Metric" (at 291.7952 195.58 0)
-      (effects (font (size 1.27 1.27)) hide)
-    )
+    (property "Footprint" "Capacitor_SMD:C_0402_1005Metric" (at 291.7952 195.58 0)
+      (effects (font (size 1.27 1.27)) hide)
+    )

Commit message: cleanded pcb directory
Parts:
- C33, C34: value 12p -> 9p
Changed lines of the file:
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@@
       (effects (font (size 1.27 1.27)))
     )
-    (property "Value" "12p" (at 60.325 140.335 90)
+    (property "Value" "9p" (at 60.325 140.335 90)
       (effects (font (size 1.27 1.27)))
     )
@@
       (effects (font (size 1.27 1.27)))
     )
-    (property "Value" "12p" (at 60.325 154.94 90)
-      (effects (font (size 1.27 1.27)))
-    )
+    (property "Value" "9p" (at 60.325 154.94 90)
+      (effects (font (size 1.27 1.27)))
+    )
